File: stack-light.kicad_pcb (KiCad board)
At the start: 2 copper layers, 132 x 60 mm, 131 parts, among them J2 Mini-DIN-6, J3 Barrel_Jack_Switch, J4 USB_C_Receptacle_USB2.0, Q1 2N7002, Q2 2N7002, Q3 2N7002, Q4 2N7002, Q6 BC817-40, Q7 BC817-40, U1 MP8007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

Commit message: Bump revision to r1.2
Also perform minor silkscreen cleanup
Other:
- board text added: "POE stack light controller r1.2"
- board text removed: "POE stack light controller r1.0"
- board text removed: "POE stack light controller r1.1"
Changed lines of the file:
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@@
     (descr "DCDC-Converter, TRACO, TSR 1-xxxx")
     (tags "DCDC-Converter TRACO TSR-1")
-    (fp_text reference U13 (at -1.5 -6.71) (layer F.SilkS)
+    (fp_text reference U13 (at -2 0 90) (layer F.SilkS)
       (effects (font (size 1 1) (thickness 0.15)))
     )
@@
       (effects (font (size 0.8 0.8) (thickness 0.12)))
     )
-    (pad 2 smd roundrect (at 1.4625 0) (size 1.125 2.65) (layers F.Cu F.Paste F.Mask) (roundrect_rratio 0.2222213333333333)
+    (pad 2 smd roundrect (at 1.4625 0) (size 1.125 2.65) (layers F.Cu F.Paste F.Mask) (roundrect_rratio 0.2222204444444444)
       (net 6 GND))
-    (pad 1 smd roundrect (at -1.4625 0) (size 1.125 2.65) (layers F.Cu F.Paste F.Mask) (roundrect_rratio 0.2222213333333333)
+    (pad 1 smd roundrect (at -1.4625 0) (size 1.125 2.65) (layers F.Cu F.Paste F.Mask) (roundrect_rratio 0.2222204444444444)
       (net 9 +12V))
     (model ${KISYS3DMOD}/Resistor_SMD.3dshapes/R_1210_3225Metric.wrl
@@
       (effects (font (size 0.8 0.8) (thickness 0.12)))
     )
-    (pad 2 smd roundrect (at 1.4625 0) (size 1.125 2.65) (layers F.Cu F.Paste F.Mask) (roundrect_rratio 0.2222213333333333)
+    (pad 2 smd roundrect (at 1.4625 0) (size 1.125 2.65) (layers F.Cu F.Paste F.Mask) (roundrect_rratio 0.2222204444444444)
       (net 6 GND))
-    (pad 1 smd roundrect (at -1.4625 0) (size 1.125 2.65) (layers F.Cu F.Paste F.Mask) (roundrect_rratio 0.2222213333333333)
+    (pad 1 smd roundrect (at -1.4625 0) (size 1.125 2.65) (layers F.Cu F.Paste F.Mask) (roundrect_rratio 0.2222204444444444)
       (net 9 +12V))
     (model ${KISYS3DMOD}/Resistor_SMD.3dshapes/R_1210_3225Metric.wrl
@@
     (tags capacitor)
     (attr smd)
-    (fp_text reference C30 (at -3.25 0 90) (layer F.SilkS)
+    (fp_text reference C30 (at -2.5 -0.25 180) (layer F.SilkS)
       (effects (font (size 1 1) (thickness 0.15)))
     )
@@
     (tags capacitor)
     (attr smd)
-    (fp_text reference C29 (at -2.975 0 90) (layer F.SilkS)
+    (fp_text reference C29 (at -2.25 -1 180) (layer F.SilkS)
       (effects (font (size 1 1) (thickness 0.15)))
     )
@@
     (tags SOT-23-5)
     (attr smd)
-    (fp_text reference U7 (at 0 2.5) (layer F.SilkS)
+    (fp_text reference U7 (at -0.35 2.5) (layer F.SilkS)
       (effects (font (size 1 1) (thickness 0.15)))
     )
@@
     (tags resistor)
     (attr smd)
-    (fp_text reference R8 (at 0 1.65) (layer B.SilkS)
+    (fp_text reference R8 (at 2.8375 0) (layer B.SilkS)
       (effects (font (size 1 1) (thickness 0.15)) (justify mirror))
     )
@@
       (effects (font (size 0.8 0.8) (thickness 0.12)))
     )
-    (pad 2 smd roundrect (at 1.4625 0 90) (size 1.125 1.75) (layers F.Cu F.Paste F.Mask) (roundrect_rratio 0.2222204444444444)
+    (pad 2 smd roundrect (at 1.4625 0 90) (size 1.125 1.75) (layers F.Cu F.Paste F.Mask) (roundrect_rratio 0.2222195555555556)
       (net 2 POE_VIN))
-    (pad 1 smd roundrect (at -1.4625 0 90) (size 1.125 1.75) (layers F.Cu F.Paste F.Mask) (roundrect_rratio 0.2222204444444444)
+    (pad 1 smd roundrect (at -1.4625 0 90) (size 1.125 1.75) (layers F.Cu F.Paste F.Mask) (roundrect_rratio 0.2222195555555556)
       (net 5 "Net-(C5-Pad2)"))
     (model ${KISYS3DMOD}/Resistor_SMD.3dshapes/R_1206_3216Metric.wrl
@@
     (tags "capacitor tantalum")
     (attr smd)
-    (fp_text reference C10 (at 0 3.1) (layer B.SilkS)
+    (fp_text reference C10 (at 0 -3.25) (layer B.SilkS)
       (effects (font (size 1 1) (thickness 0.15)) (justify mirror))
     )
@@
     (tags resistor)
     (attr smd)
-    (fp_text reference R26 (at 3.25 0) (layer F.SilkS)
+    (fp_text reference R26 (at 1.5 1.75) (layer F.SilkS)
       (effects (font (size 1 1) (thickness 0.15)))
     )
@@
     (tags capacitor)
     (attr smd)
-    (fp_text reference C7 (at 0 1.43) (layer B.SilkS)
+    (fp_text reference C7 (at -2.5375 0) (layer B.SilkS)
       (effects (font (size 1 1) (thickness 0.15)) (justify mirror))
     )
@@
   (gr_circle (center 197.1 89) (end 197.1 87.4) (layer Edge.Cuts) (width 0.2))
   (gr_line (start 205.5 108) (end 186 108) (layer Edge.Cuts) (width 0.2))
-  (gr_text "POE stack light\ncontroller r1.0" (at 162.25 85.5) (layer F.Mask)
+  (gr_text "POE stack light\ncontroller r1.2" (at 162.25 85.5) (layer F.Mask)
     (effects (font (size 1.2 1.2) (thickness 0.3)))
   )
-  (gr_text "POE stack light\ncontroller r1.1" (at 162.25 85.5) (layer F.Cu)
+  (gr_text "POE stack light\ncontroller r1.2" (at 162.25 85.5) (layer F.Cu)
     (effects (font (size 1.2 1.2) (thickness 0.3)))
   )
